File: Envelope.kicad_pcb (KiCad board)
At the start: 2 copper layers, 39.5 x 100 mm, 81 parts, among them J1 Conn_02x05_Odd_Even, J2 Conn_02x03_Odd_Even, J3 Conn_01x03, SW1 SW_SPDT_MSM, SW2 SW_SPDT_MSM, SW3 SW_Push, U1 TL072, U2 ATmega328PB-AU, U3 L7805, Y1 20MHz

Commit message: Connect CV TN to ground to avoid drift.
Connections:
- J-CV1 pad TN: Net-(J-CV1-PadTN) -> GND
